File: pcb/nt7538/evoke.sch (KiCad schematic (older format))
At the start: 40 parts, among them J1 Conn_01x03_Male, J2 BACKLIGHT_CONN, J3 SUPP_PWR, Q1 Q_NMOS_GSD, U1 STM32F103C8Tx

Commit message: NT7538 to manufacture
Parts:
- R2: value 500R -> 1K; LCSC (none) -> C17513
- R4: LCSC (none) -> C17539
Connections:
- net +3V3: now also LCD_CONN1.10 (Pin_10), LCD_CONN1.11 (Pin_11), LCD_CONN1.14 (Pin_14), LCD_CONN1.30 (Pin_30), LCD_CONN1.4 (Pin_4), LCD_CONN1.5 (Pin_5), LCD_CONN1.6 (Pin_6), LCD_CONN1.7 (Pin_7), LCD_CONN1.8 (Pin_8), LCD_CONN1.9 (Pin_9); no longer LCD_CONN1.1 (Pin_1), LCD_CONN1.17 (Pin_17), LCD_CONN1.20 (Pin_20), LCD_CONN1.21 (Pin_21), LCD_CONN1.22 (Pin_22), LCD_CONN1.23 (Pin_23), LCD_CONN1.24 (Pin_24), LCD_CONN1.25 (Pin_25), LCD_CONN1.26 (Pin_26), LCD_CONN1.27 (Pin_27)
- net GND: now also LCD_CONN1.15 (Pin_15), LCD_CONN1.28 (Pin_28), LCD_CONN1.29 (Pin_29); no longer LCD_CONN1.16 (Pin_16), LCD_CONN1.2 (Pin_2), LCD_CONN1.3 (Pin_3)
- net LCD_CS: now also LCD_CONN1.1 (Pin_1); no longer LCD_CONN1.30 (Pin_30)
- net LCD_DATA: now also LCD_CONN1.13 (Pin_13); no longer LCD_CONN1.18 (Pin_18)
- net LCD_D_C: now also LCD_CONN1.3 (Pin_3); no longer LCD_CONN1.28 (Pin_28)
- net LCD_RST: now also LCD_CONN1.2 (Pin_2); no longer LCD_CONN1.29 (Pin_29)
- net LCD_SCK: now also LCD_CONN1.12 (Pin_12); no longer LCD_CONN1.19 (Pin_19)
- net at C14.2: now also LCD_CONN1.21 (Pin_21); no longer LCD_CONN1.10 (Pin_10)
- net at C14.1: now also LCD_CONN1.20 (Pin_20); no longer LCD_CONN1.11 (Pin_11)
- net at C10.1: now also LCD_CONN1.19 (Pin_19); no longer LCD_CONN1.12 (Pin_12)
- net at C10.2, C11.2: now also LCD_CONN1.18 (Pin_18); no longer LCD_CONN1.13 (Pin_13)
- net at C11.1: now also LCD_CONN1.17 (Pin_17); no longer LCD_CONN1.14 (Pin_14)
- net at C1.1: now also LCD_CONN1.16 (Pin_16); no longer LCD_CONN1.15 (Pin_15)
- net at C15.1: now also LCD_CONN1.26 (Pin_26); no longer LCD_CONN1.5 (Pin_5)
- net at C16.1: now also LCD_CONN1.25 (Pin_25); no longer LCD_CONN1.6 (Pin_6)
- net at C17.1: now also LCD_CONN1.24 (Pin_24); no longer LCD_CONN1.7 (Pin_7)
- net at C18.1: now also LCD_CONN1.23 (Pin_23); no longer LCD_CONN1.8 (Pin_8)
- net at C19.1: now also LCD_CONN1.22 (Pin_22); no longer LCD_CONN1.9 (Pin_9)
Changed lines of the file:
@@
 SDIN_IN
-$Comp
-L evoke-rescue:Conn_01x30-Connector_Generic-evoke-rescue LCD_CONN1
-U 1 1 5EA08ED1
-P 2750 4550
-F 0 "LCD_CONN1" V 2967 4496 50  0000 C CNN
-F 1 "Conn_01x30" V 2876 4496 50  0000 C CNN
-F 2 "Connector_FFC-FPC:Hirose_FH12-30S-0.5SH_1x30-1MP_P0.50mm_Horizontal" H 2750 4550 50  0001 C CNN
-F 3 "~" H 2750 4550 50  0001 C CNN
-	1    2750 4550
-	0    -1   -1   0
-$EndComp
 $Comp
 L evoke-rescue:+3V3-power-evoke-rescue #PWR0106
@@
 P 5050 6650
 F 0 "R2" V 4843 6650 50  0000 C CNN
-F 1 "500R" V 4934 6650 50  0000 C CNN
+F 1 "1K" V 4934 6650 50  0000 C CNN
 F 2 "Resistor_SMD:R_0805_2012Metric" V 4980 6650 50  0001 C CNN
 F 3 "" H 5050 6650 50  0001 C CNN
+F 4 "C17513" V 5050 6650 50  0001 C CNN "LCSC"
 	1    5050 6650
 	0    1    1    0
@@
 F 2 "Resistor_SMD:R_0805_2012Metric" V 5130 6800 50  0001 C CNN
 F 3 "" H 5200 6800 50  0001 C CNN
+F 4 "C17539" H 5200 6800 50  0001 C CNN "LCSC"
 	1    5200 6800
 	1    0    0    -1
@@
 	1500 4750 1550 4750
 Connection ~ 1500 4750
+$Comp
+L evoke-rescue:Conn_01x30-Connector_Generic-evoke-rescue LCD_CONN1
+U 1 1 5EA08ED1
+P 2850 4550
+F 0 "LCD_CONN1" V 3067 4496 50  0000 C CNN
+F 1 "Conn_01x30" V 2976 4496 50  0000 C CNN
+F 2 "Connector_FFC-FPC:Hirose_FH12-30S-0.5SH_1x30-1MP_P0.50mm_Horizontal" H 2850 4550 50  0001 C CNN
+F 3 "~" H 2850 4550 50  0001 C CNN
+	1    2850 4550
+	0    1    -1   0
+$EndComp
 $EndSCHEMATC
